File: Hardware/dish-controller/dish-controller.kicad_pcb (KiCad board)
At the start: 4 copper layers, 165 x 70 mm, 53 parts, among them J1 12V-IN, J2 5V-IN, J3 Encoder_Conn, J4 Encoder_Conn, J5 AZ-OUT, J6 EL-OUT, Q5 BSS138, Q6 BSS138, Q7 BSS138, Q8 BSS138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

Commit message: Dish Controller: Update 3D Model
Added models for the raspberry pi and heatsinks.
Parts:
- added H1: MountingHole, MountingHole:MountingHole_3.2mm_M3, F.Cu at (41.0, 75.0)
- moved C1 3.54 mm to (81.5, 84.8)
- moved G1 2.50 mm to (173.0, 103.5)
Connections:
- U1 pad 16: unconnected-(U1-Pad16) -> /EPWM1
- U1 pad 18: unconnected-(U1-Pad18) -> /EPWM2
Routing:
- net /EPWM2: track 2.05 -> 49.2 mm, vias 0 -> 1
- net /EPWM1: track 2.11 -> 47.4 mm, vias 0 -> 1
- net GND: track 78.6 -> 114.6 mm, vias 18 -> 19
- net +12V: track 50.3 -> 73.3 mm
- net /A22: track 116.9 -> 130.8 mm
- net /A21: track 81.5 -> 83.0 mm
Other:
- board text added: "12V"
- board text added: "5V"
- board text added: "AZ"
- board text added: "CLK"
- board text added: "Designed by Hans Gaensbauer and Eli Reed"
- board text added: "EL"
- board text added: "ETHERNET"
- board text added: "GND"
- board text added: "IN11"
- board text added: "IN21"
- board text added: "IN22"
- board text added: "Interferometer Dish Controller Rev 0"
- board text added: "Radio Astronomy at the Speed of Light"
- board text added: "SDI"
- board text added: "SDO"
- board text added: "~{CS}1"
- board text added: "~{CS}2"
