File: Hardware/dish-controller/level-shift.kicad_sch (KiCad schematic)
At the start: 12 parts, among them Q1 BSS138, Q2 BSS138, Q3 BSS138, Q4 BSS138

Commit message: Dish Control: DRC Pass
Floorplanning and routing for dish control PCB complete
Parts:
- R19: renamed from R11; footprint (none) -> Resistor_SMD:R_0603_1608Metric
- R20: renamed from R12; footprint (none) -> Resistor_SMD:R_0603_1608Metric
- R21: renamed from R13; footprint (none) -> Resistor_SMD:R_0603_1608Metric
- R22: renamed from R14; footprint (none) -> Resistor_SMD:R_0603_1608Metric
- R23: renamed from R15; footprint (none) -> Resistor_SMD:R_0603_1608Metric
- R24: renamed from R16; footprint (none) -> Resistor_SMD:R_0603_1608Metric
- R25: renamed from R17; footprint (none) -> Resistor_SMD:R_0603_1608Metric
- R26: renamed from R18; footprint (none) -> Resistor_SMD:R_0603_1608Metric
- renumbered Q1 to Q5, Q2 to Q6, Q3 to Q7, Q4 to Q8
Changed lines of the file:
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@@
   (symbol (lib_id "Device:R_Small") (at 132.08 109.22 180)
     (in_bom yes) (on_board yes)
-    (property "Reference" "R18" (id 0) (at 129.54 107.95 0))
+    (property "Reference" "R26" (id 0) (at 129.54 107.95 0))
     (property "Value" "10k" (id 1) (at 129.54 110.49 0))
-    (property "Footprint" "" (id 2) (at 132.08 109.22 0)
+    (property "Footprint" "Resistor_SMD:R_0603_1608Metric" (id 2) (at 132.08 109.22 0)
       (effects (font (size 1.27 1.27)) hide)
     )
@@
   (symbol (lib_id "Transistor_FET:BSS138") (at 123.19 88.9 270)
     (in_bom yes) (on_board yes) (fields_autoplaced)
-    (property "Reference" "Q3" (id 0) (at 123.19 95.4945 90))
+    (property "Reference" "Q7" (id 0) (at 123.19 95.4945 90))
     (property "Value" "BSS138" (id 1) (at 123.19 98.2696 90))
     (property "Footprint" "Package_TO_SOT_SMD:SOT-23" (id 2) (at 121.285 93.98 0)
@@
   (symbol (lib_id "Device:R_Small") (at 114.3 86.36 180)
     (in_bom yes) (on_board yes)
-    (property "Reference" "R15" (id 0) (at 111.76 85.09 0))
+    (property "Reference" "R23" (id 0) (at 111.76 85.09 0))
     (property "Value" "10k" (id 1) (at 111.76 87.63 0))
-    (property "Footprint" "" (id 2) (at 114.3 86.36 0)
+    (property "Footprint" "Resistor_SMD:R_0603_1608Metric" (id 2) (at 114.3 86.36 0)
       (effects (font (size 1.27 1.27)) hide)
     )
@@
   (symbol (lib_id "Device:R_Small") (at 132.08 86.36 180)
     (in_bom yes) (on_board yes)
-    (property "Reference" "R17" (id 0) (at 129.54 85.09 0))
+    (property "Reference" "R25" (id 0) (at 129.54 85.09 0))
     (property "Value" "10k" (id 1) (at 129.54 87.63 0))
-    (property "Footprint" "" (id 2) (at 132.08 86.36 0)
+    (property "Footprint" "Resistor_SMD:R_0603_1608Metric" (id 2) (at 132.08 86.36 0)
       (effects (font (size 1.27 1.27)) hide)
     )
@@
   (symbol (lib_id "Device:R_Small") (at 76.2 86.36 180)
     (in_bom yes) (on_board yes)
-    (property "Reference" "R11" (id 0) (at 73.66 85.09 0))
+    (property "Reference" "R19" (id 0) (at 73.66 85.09 0))
     (property "Value" "10k" (id 1) (at 73.66 87.63 0))
-    (property "Footprint" "" (id 2) (at 76.2 86.36 0)
+    (property "Footprint" "Resistor_SMD:R_0603_1608Metric" (id 2) (at 76.2 86.36 0)
       (effects (font (size 1.27 1.27)) hide)
     )
@@
   (symbol (lib_id "Device:R_Small") (at 114.3 109.22 180)
     (in_bom yes) (on_board yes)
-    (property "Reference" "R16" (id 0) (at 111.76 107.95 0))
+    (property "Reference" "R24" (id 0) (at 111.76 107.95 0))
     (property "Value" "10k" (id 1) (at 111.76 110.49 0))
-    (property "Footprint" "" (id 2) (at 114.3 109.22 0)
+    (property "Footprint" "Resistor_SMD:R_0603_1608Metric" (id 2) (at 114.3 109.22 0)
       (effects (font (size 1.27 1.27)) hide)
     )
@@
   (symbol (lib_id "Device:R_Small") (at 93.98 86.36 180)
     (in_bom yes) (on_board yes)
-    (property "Reference" "R13" (id 0) (at 91.44 85.09 0))
+    (property "Reference" "R21" (id 0) (at 91.44 85.09 0))
     (property "Value" "10k" (id 1) (at 91.44 87.63 0))
-    (property "Footprint" "" (id 2) (at 93.98 86.36 0)
+    (property "Footprint" "Resistor_SMD:R_0603_1608Metric" (id 2) (at 93.98 86.36 0)
       (effects (font (size 1.27 1.27)) hide)
     )
@@
   (symbol (lib_id "Device:R_Small") (at 93.98 109.22 180)
     (in_bom yes) (on_board yes)
-    (property "Reference" "R14" (id 0) (at 91.44 107.95 0))
+    (property "Reference" "R22" (id 0) (at 91.44 107.95 0))
     (property "Value" "10k" (id 1) (at 91.44 110.49 0))
-    (property "Footprint" "" (id 2) (at 93.98 109.22 0)
+    (property "Footprint" "Resistor_SMD:R_0603_1608Metric" (id 2) (at 93.98 109.22 0)
       (effects (font (size 1.27 1.27)) hide)
     )
@@
   (symbol (lib_id "Transistor_FET:BSS138") (at 85.09 111.76 270)
     (in_bom yes) (on_board yes) (fields_autoplaced)
-    (property "Reference" "Q2" (id 0) (at 85.09 118.3545 90))
+    (property "Reference" "Q6" (id 0) (at 85.09 118.3545 90))
     (property "Value" "BSS138" (id 1) (at 85.09 121.1296 90))
     (property "Footprint" "Package_TO_SOT_SMD:SOT-23" (id 2) (at 83.185 116.84 0)
@@
   (symbol (lib_id "Transistor_FET:BSS138") (at 85.09 88.9 270)
     (in_bom yes) (on_board yes) (fields_autoplaced)
-    (property "Reference" "Q1" (id 0) (at 85.09 95.4945 90))
+    (property "Reference" "Q5" (id 0) (at 85.09 95.4945 90))
     (property "Value" "BSS138" (id 1) (at 85.09 98.2696 90))
     (property "Footprint" "Package_TO_SOT_SMD:SOT-23" (id 2) (at 83.185 93.98 0)
@@
   (symbol (lib_id "Transistor_FET:BSS138") (at 123.19 111.76 270)
     (in_bom yes) (on_board yes) (fields_autoplaced)
-    (property "Reference" "Q4" (id 0) (at 123.19 118.3545 90))
+    (property "Reference" "Q8" (id 0) (at 123.19 118.3545 90))
     (property "Value" "BSS138" (id 1) (at 123.19 121.1296 90))
     (property "Footprint" "Package_TO_SOT_SMD:SOT-23" (id 2) (at 121.285 116.84 0)
@@
   (symbol (lib_id "Device:R_Small") (at 76.2 109.22 180)
     (in_bom yes) (on_board yes)
-    (property "Reference" "R12" (id 0) (at 73.66 107.95 0))
+    (property "Reference" "R20" (id 0) (at 73.66 107.95 0))
     (property "Value" "10k" (id 1) (at 73.66 110.49 0))
-    (property "Footprint" "" (id 2) (at 76.2 109.22 0)
-      (effects (font (size 1.27 1.27)) hide)
-    )
+    (property "Footprint" "Resistor_SMD:R_0603_1608Metric" (id 2) (at 76.2 109.22 0)
+      (effects (font (size 1.27 1.27)) hide)
+    )

Commit message: Dish Controller: Plot
Parts:
- Q5, Q6, Q7, Q8: footprint Package_TO_SOT_SMD:SOT-23 -> Package_TO_SOT_SMD:SOT-323_SC-70
Changed lines of the file:
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@@
     (property "Reference" "Q7" (id 0) (at 123.19 95.4945 90))
     (property "Value" "BSS138" (id 1) (at 123.19 98.2696 90))
-    (property "Footprint" "Package_TO_SOT_SMD:SOT-23" (id 2) (at 121.285 93.98 0)
+    (property "Footprint" "Package_TO_SOT_SMD:SOT-323_SC-70" (id 2) (at 121.285 93.98 0)
       (effects (font (size 1.27 1.27) italic) (justify left) hide)
     )
@@
     (property "Reference" "Q6" (id 0) (at 85.09 118.3545 90))
     (property "Value" "BSS138" (id 1) (at 85.09 121.1296 90))
-    (property "Footprint" "Package_TO_SOT_SMD:SOT-23" (id 2) (at 83.185 116.84 0)
+    (property "Footprint" "Package_TO_SOT_SMD:SOT-323_SC-70" (id 2) (at 83.185 116.84 0)
       (effects (font (size 1.27 1.27) italic) (justify left) hide)
     )
@@
     (property "Reference" "Q5" (id 0) (at 85.09 95.4945 90))
     (property "Value" "BSS138" (id 1) (at 85.09 98.2696 90))
-    (property "Footprint" "Package_TO_SOT_SMD:SOT-23" (id 2) (at 83.185 93.98 0)
+    (property "Footprint" "Package_TO_SOT_SMD:SOT-323_SC-70" (id 2) (at 83.185 93.98 0)
       (effects (font (size 1.27 1.27) italic) (justify left) hide)
     )
@@
     (property "Reference" "Q8" (id 0) (at 123.19 118.3545 90))
     (property "Value" "BSS138" (id 1) (at 123.19 121.1296 90))
-    (property "Footprint" "Package_TO_SOT_SMD:SOT-23" (id 2) (at 121.285 116.84 0)
-      (effects (font (size 1.27 1.27) italic) (justify left) hide)
-    )
+    (property "Footprint" "Package_TO_SOT_SMD:SOT-323_SC-70" (id 2) (at 121.285 116.84 0)
+      (effects (font (size 1.27 1.27) italic) (justify left) hide)
+    )
